File: KiCad/esp32_s3_weather_webserver.kicad_sch (KiCad schematic)
At the start: 1 part, among them IC101 ESP32-S3-WROOM-1-N16R8

Commit message: USB scheme
Parts:
- removed IC101: ESP32-S3-WROOM-1-N16R8, esp32_s3_weather_webserver:ESP32S3WROOM1N16R8, symbol esp32_s3_weather_webserver:ESP32-S3-WROOM-1-N16R8
Other:
- added sheet [2] Power (02_power.kicad_sch)
- added sheet [3] USB (03_usb.kicad_sch)
- added sheet [4] ESP32 S3 (04_esp32_s3.kicad_sch)
- added sheet [5] Peripherals (05_peripherals.kicad_sch)
Changed lines of the file:
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@@
 	(generator_version "9.0")
 	(paper "A4")
-	(symbol
-		(lib_id "esp32_s3_weather_webserver:ESP32-S3-WROOM-1-N16R8")
-		(at 52.07 53.34 0)
-		(unit 1)
+	(sheet
+		(at 63.5 38.1)
+		(size 25.4 25.4)
 		(exclude_from_sim no)
 		(in_bom yes)
@@
 		(dnp no)
 		(fields_autoplaced yes)
-		(property "Reference" "IC101"
-			(at 66.04 127 0)
+		(stroke
+			(width 0.1524)
+			(type solid)
+		)
+		(fill
+			(color 0 0 0 0.0000)
+		)
+		(property "Sheetname" "[3] USB"
+			(at 63.5 37.3884 0)
 			(effects
 				(font
 					(size 1.27 1.27)
 				)
+				(justify left bottom)
 			)
 		)
-		(property "Value" "ESP32-S3-WROOM-1-N16R8"
-			(at 66.04 129.54 0)
-			(effects
-				(font
-					(size 1.27 1.27)
-				)
-			)
-		)
-		(property "Footprint" "esp32_s3_weather_webserver:ESP32S3WROOM1N16R8"
-			(at 81.28 148.26 0)
+		(property "Sheetfile" "03_usb.kicad_sch"
+			(at 63.5 64.0846 0)
 			(effects
 				(font
@@
 				)
 				(justify left top)
-				(hide yes)
 			)
 		)
-		(property "Datasheet" "https://www.espressif.com/sites/default/files/documentation/esp32-s3-wroom-1_wroom-1u_datasheet_en.pdf"
-			(at 81.28 248.26 0)
+		(instances
+			(project "esp32_s3_weather_webserver"
+				(path "/04e96486-ec4c-4881-a0bf-37cb6ce91c2d"
+					(page "3")
+				)
+			)
+		)
+	)
+	(sheet
+		(at 101.6 38.1)
+		(size 25.4 25.4)
+		(exclude_from_sim no)
+		(in_bom yes)
+		(on_board yes)
+		(dnp no)
+		(fields_autoplaced yes)
+		(stroke
+			(width 0.1524)
+			(type solid)
+		)
+		(fill
+			(color 0 0 0 0.0000)
+		)
+		(property "Sheetname" "[4] ESP32 S3"
+			(at 101.6 37.3884 0)
+			(effects
+				(font
+					(size 1.27 1.27)
+				)
+				(justify left bottom)
+			)
+		)
+		(property "Sheetfile" "04_esp32_s3.kicad_sch"
+			(at 101.6 64.0846 0)
 			(effects
 				(font
@@
 				)
 				(justify left top)
-				(hide yes)
 			)
 		)
-		(property "Description" "Multiprotocol Modules SMD Module, ESP32-S3R8, 3.3V, 8 MB Octal PSRAM Die, 16 MB Quad SPI Flash, PCB Antenna"
-			(at 63.246 165.1 0)
+		(instances
+			(project "esp32_s3_weather_webserver"
+				(path "/04e96486-ec4c-4881-a0bf-37cb6ce91c2d"
+					(page "4")
+				)
+			)
+		)
+	)
+	(sheet
+		(at 25.4 38.1)
+		(size 25.4 25.4)
+		(exclude_from_sim no)
+		(in_bom yes)
+		(on_board yes)
+		(dnp no)
+		(fields_autoplaced yes)
+		(stroke
+			(width 0.1524)
+			(type solid)
+		)
+		(fill
+			(color 0 0 0 0.0000)
+		)
+		(property "Sheetname" "[2] Power"
+			(at 25.4 37.3884 0)
 			(effects
 				(font
 					(size 1.27 1.27)
 				)
-				(hide yes)
+				(justify left bottom)
 			)
 		)
-		(property "Height" "3.25"
-			(at 81.28 448.26 0)
+		(property "Sheetfile" "02_power.kicad_sch"
+			(at 25.4 64.0846 0)
 			(effects
 				(font
@@
 				)
 				(justify left top)
-				(hide yes)
 			)
 		)
-		(property "Manufacturer_Name" "Espressif Systems"
-			(at 81.28 548.26 0)
+		(instances
+			(project "esp32_s3_weather_webserver"
+				(path "/04e96486-ec4c-4881-a0bf-37cb6ce91c2d"
+					(page "2")
+				)
+			)
+		)
+	)
+	(sheet
+		(at 139.7 38.1)
+		(size 25.4 25.4)
+		(exclude_from_sim no)
+		(in_bom yes)
+		(on_board yes)
+		(dnp no)
+		(fields_autoplaced yes)
+		(stroke
+			(width 0.1524)
+			(type solid)
+		)
+		(fill
+			(color 0 0 0 0.0000)
+		)
+		(property "Sheetname" "[5] Peripherals"
+			(at 139.7 37.3884 0)
+			(effects
+				(font
+					(size 1.27 1.27)
+				)
+				(justify left bottom)
+			)
+		)
+		(property "Sheetfile" "05_peripherals.kicad_sch"
+			(at 139.7 64.0846 0)
 			(effects
 				(font
@@
 				)
 				(justify left top)
-				(hide yes)
 			)
 		)
-		(property "Manufacturer_Part_Number" "ESP32-S3-WROOM-1-N16R8"
-			(at 81.28 648.26 0)
-			(effects
-				(font
-					(size 1.27 1.27)
-				)
-				(justify left top)
-				(hide yes)
-			)
-		)
-		(property "Mouser Part Number" "356-ESP32S3WRM1N16R8"
-			(at 81.28 748.26 0)
-			(effects
-				(font
-					(size 1.27 1.27)
-				)
-				(justify left top)
-				(hide yes)
-			)
-		)
-		(property "Mouser Price/Stock" "https://www.mouser.co.uk/ProductDetail/Espressif-Systems/ESP32-S3-WROOM-1-N16R8?qs=Li%252BoUPsLEnvQc9gW6AMhZg%3D%3D"
-			(at 81.28 848.26 0)
-			(effects
-				(font
-					(size 1.27 1.27)
-				)
-				(justify left top)
-				(hide yes)
-			)
-		)
-		(property "Arrow Part Number" ""
-			(at 81.28 948.26 0)
-			(effects
-				(font
-					(size 1.27 1.27)
-				)
-				(justify left top)
-				(hide yes)
-			)
-		)
-		(property "Arrow Price/Stock" ""
-			(at 81.28 1048.26 0)
-			(effects
-				(font
-					(size 1.27 1.27)
-				)
-				(justify left top)
-				(hide yes)
-			)
-		)
-		(pin "33"
-		)
-		(pin "28"
-		)
-		(pin "31"
-		)
-		(pin "48"
-		)
-		(pin "23"
-		)
-		(pin "8"
-		)
-		(pin "26"
-		)
-		(pin "44"
-		)
-		(pin "29"
-		)
-		(pin "47"
-		)
-		(pin "30"
-		)
-		(pin "41"
-		)
-		(pin "25"
-		)
-		(pin "46"
-		)
-		(pin "14"
-		)
-		(pin "24"
-		)
-		(pin "5"
-		)
-		(pin "34"
-		)
-		(pin "9"
-		)
-		(pin "2"
-		)
-		(pin "21"
-		)
-		(pin "43"
-		)
-		(pin "49"
-		)
-		(pin "32"
-		)
-		(pin "17"
-		)
-		(pin "6"
-		)
-		(pin "13"
-		)
-		(pin "10"
-		)
-		(pin "11"
-		)
-		(pin "40"
-		)
-		(pin "16"
-		)
-		(pin "4"
-		)
-		(pin "19"
-		)
-		(pin "7"
-		)
-		(pin "22"
-		)
-		(pin "18"
-		)
-		(pin "20"
-		)
-		(pin "35"
-		)
-		(pin "1"
-		)
-		(pin "42"
-		)
-		(pin "12"
-		)
-		(pin "37"
-		)
-		(pin "45"
-		)
-		(pin "15"
-		)
-		(pin "3"
-		)
-		(pin "27"
-		)
-		(pin "38"
-		)
-		(pin "36"
-		)
-		(pin "39"
-		)
 		(instances
-			(project ""
+			(project "esp32_s3_weather_webserver"
 				(path "/04e96486-ec4c-4881-a0bf-37cb6ce91c2d"
-					(reference "IC101")
-					(unit 1)
+					(page "5")
 				)
 			)

Commit message: BOM updates
Parts:
- added H1, H2, H3, H4: MountingHole, MountingHole:MountingHole_3.2mm_M3, symbol Mechanical:MountingHole
Other:
- note added: "Mounting Holes (M3)"

Commit message: BOM updates. First layout
Parts:
- renumbered H1 to H101, H2 to H102, H3 to H103, H4 to H104
Changed lines of the file:
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@@
 		(dnp no)
 		(fields_autoplaced yes)
-		(property "Reference" "H1"
+		(property "Reference" "H101"
 			(at 20.32 172.7199 0)
 			(effects
@@
 			(project "esp32_s3_weather_webserver"
 				(path "/04e96486-ec4c-4881-a0bf-37cb6ce91c2d"
-					(reference "H1")
+					(reference "H101")
 					(unit 1)
 				)
@@
 		(dnp no)
 		(fields_autoplaced yes)
-		(property "Reference" "H4"
+		(property "Reference" "H104"
 			(at 20.32 191.7699 0)
 			(effects
@@
 			(project "esp32_s3_weather_webserver"
 				(path "/04e96486-ec4c-4881-a0bf-37cb6ce91c2d"
-					(reference "H4")
+					(reference "H104")
 					(unit 1)
 				)
@@
 		(dnp no)
 		(fields_autoplaced yes)
-		(property "Reference" "H3"
+		(property "Reference" "H103"
 			(at 20.32 185.4199 0)
 			(effects
@@
 			(project "esp32_s3_weather_webserver"
 				(path "/04e96486-ec4c-4881-a0bf-37cb6ce91c2d"
-					(reference "H3")
+					(reference "H103")
 					(unit 1)
 				)
@@
 		(dnp no)
 		(fields_autoplaced yes)
-		(property "Reference" "H2"
+		(property "Reference" "H102"
 			(at 20.32 179.0699 0)
 			(effects
@@
 			(project "esp32_s3_weather_webserver"
 				(path "/04e96486-ec4c-4881-a0bf-37cb6ce91c2d"
-					(reference "H2")
-					(unit 1)
-				)
+					(reference "H102")
+					(unit 1)
+				)
